File: KeyGrid_Right.kicad_sch (KiCad schematic)
At the start: 76 parts, among them SW10 SW_Push_45deg, SW11 SW_Push_45deg, SW12 SW_Push_45deg, SW13 SW_Push_45deg, SW14 SW_Push_45deg, SW15 SW_Push_45deg, SW16 SW_Push_45deg, SW17 SW_Push_45deg, SW18 SW_Push_45deg, SW19 SW_Push_45deg, SW20 SW_Push_45deg, SW21 SW_Push_45deg, SW22 SW_Push_45deg, SW23 SW_Push_45deg, SW24 SW_Push_45deg, SW25 SW_Push_45deg, SW26 SW_Push_45deg, SW27 SW_Push_45deg, SW29 SW_Push_45deg, SW30 SW_Push_45deg, SW31 SW_Push_45deg, SW32 SW_Push_45deg, SW33 SW_Push_45deg, SW34 SW_Push_45deg, SW35 SW_Push_45deg, SW36 SW_Push_45deg, SW37 SW_Push_45deg, SW38 SW_Push_45deg, SW39 SW_Push_45deg, SW40 SW_Push_45deg, SW41 SW_Push_45deg, SW42 SW_Push_45deg, SW43 SW_Push_45deg, SW5 SW_Push_45deg, SW6 SW_Push_45deg, SW7 SW_Push_45deg, SW8 SW_Push_45deg, SW9 SW_Push_45deg

Commit message: Added footprints and started PCB layout
Parts:
- removed D39, D40, D41, D42, D43: 1N4148WT, Diode_SMD:D_SOD-123, symbol Diode:1N4148WT
- removed SW39, SW40, SW41, SW42, SW43: SW_Push_45deg, PCM_Switch_Keyboard_Hotswap_Kailh:SW_Hotswap_Kailh_Choc_V1V2_1.00u, symbol Switch:SW_Push_45deg
- SW10, SW16: footprint PCM_Switch_Keyboard_Hotswap_Kailh:SW_Hotswap_Kailh_Choc_V1V2_1.25u -> Button_Switch_Keyboard:SW_Cherry_MX_1.00u_PCB
- SW11, SW12, SW13, SW14, SW15, SW17, SW18, SW19, SW20, SW21, SW23, SW24, SW25, SW26, SW27, SW29, SW30, SW31, SW32, SW33, SW34, SW35, SW36, SW37, SW38, SW5, SW6, SW7, SW8, SW9: footprint PCM_Switch_Keyboard_Hotswap_Kailh:SW_Hotswap_Kailh_Choc_V1V2_1.00u -> Button_Switch_Keyboard:SW_Cherry_MX_1.00u_PCB
- SW22: footprint PCM_Switch_Keyboard_Hotswap_Kailh:SW_Hotswap_Kailh_Choc_V1V2_1.50u -> Button_Switch_Keyboard:SW_Cherry_MX_1.00u_PCB
