File: Keybrd_Part_2.kicad_pcb (KiCad board)
At the start: 2 copper layers, 121 parts, among them SW2 SW_Push, SW3 SW_Push, SW4 SW_Push, U1 RP2040, U2 AP2112K-3.3, U4 W25Q128JVS, U5 W25Q128JVS, U6 RP2040, Y1 12MHz Crystal GND24, Y2 12MHz Crystal GND24

Commit message: Added footprints and started PCB layout
Parts:
- removed D39, D40, D41, D42, D43: 1N4148WT, Diode_SMD:D_SOD-123
- added J3: USB_C_Receptacle_USB2.0_14P, Connector_USB:USB_C_Receptacle_GCT_USB4125-xx-x-0190_6P_TopMnt_Horizontal, F.Cu at (235.9, 93.0)
- added J5: USB_C_Receptacle_USB2.0_14P, Connector_USB:USB_C_Receptacle_GCT_USB4125-xx-x-0190_6P_TopMnt_Horizontal, F.Cu at (226.0, 108.2)
- added J7: USB_C_Receptacle_USB2.0_14P, Connector_USB:USB_C_Receptacle_GCT_USB4125-xx-x-0190_6P_TopMnt_Horizontal, F.Cu at (185.6, 108.1)
- added SW1: SW_Push_45deg, Button_Switch_Keyboard:SW_Cherry_MX_1.00u_PCB, F.Cu at (129.4, 187.7)
- added SW10: SW_Push_45deg, Button_Switch_Keyboard:SW_Cherry_MX_1.00u_PCB, F.Cu at (242.2, 197.7)
- added SW11: SW_Push_45deg, Button_Switch_Keyboard:SW_Cherry_MX_1.00u_PCB, F.Cu at (281.1, 91.1)
- added SW12: SW_Push_45deg, Button_Switch_Keyboard:SW_Cherry_MX_1.00u_PCB, F.Cu at (281.1, 110.1)
- added SW13: SW_Push_45deg, Button_Switch_Keyboard:SW_Cherry_MX_1.00u_PCB, F.Cu at (281.1, 129.1)
- added SW14: SW_Push_45deg, Button_Switch_Keyboard:SW_Cherry_MX_1.00u_PCB, F.Cu at (281.1, 148.1)
- added SW15: SW_Push_45deg, Button_Switch_Keyboard:SW_Cherry_MX_1.00u_PCB, F.Cu at (281.1, 167.0)
- added SW16: SW_Push_45deg, Button_Switch_Keyboard:SW_Cherry_MX_1.00u_PCB, F.Cu at (264.6, 192.0)
- added SW17: SW_Push_45deg, Button_Switch_Keyboard:SW_Cherry_MX_1.00u_PCB, F.Cu at (300.1, 85.1)
- added SW18: SW_Push_45deg, Button_Switch_Keyboard:SW_Cherry_MX_1.00u_PCB, F.Cu at (300.1, 104.1)
- added SW19: SW_Push_45deg, Button_Switch_Keyboard:SW_Cherry_MX_1.00u_PCB, F.Cu at (300.1, 123.1)
- added SW20: SW_Push_45deg, Button_Switch_Keyboard:SW_Cherry_MX_1.00u_PCB, F.Cu at (300.1, 142.1)
- added SW21: SW_Push_45deg, Button_Switch_Keyboard:SW_Cherry_MX_1.00u_PCB, F.Cu at (300.2, 161.0)
- added SW22: SW_Push_45deg, Button_Switch_Keyboard:SW_Cherry_MX_1.00u_PCB, F.Cu at (287.5, 189.5)
- added SW23: SW_Push_45deg, Button_Switch_Keyboard:SW_Cherry_MX_1.00u_PCB, F.Cu at (319.2, 92.1)
- added SW24: SW_Push_45deg, Button_Switch_Keyboard:SW_Cherry_MX_1.00u_PCB, F.Cu at (319.1, 111.1)
- added SW25: SW_Push_45deg, Button_Switch_Keyboard:SW_Cherry_MX_1.00u_PCB, F.Cu at (319.1, 130.1)
- added SW26: SW_Push_45deg, Button_Switch_Keyboard:SW_Cherry_MX_1.00u_PCB, F.Cu at (319.1, 149.0)
- added SW27: SW_Push_45deg, Button_Switch_Keyboard:SW_Cherry_MX_1.00u_PCB, F.Cu at (319.1, 168.1)
- added SW28: SW_Push, PTS636_SM43J_SMTR_LFS:SW_PTS636_SM43J_SMTR_LFS, F.Cu at (215.4, 159.6)
- added SW29: SW_Push_45deg, Button_Switch_Keyboard:SW_Cherry_MX_1.00u_PCB, F.Cu at (338.2, 104.1)
- added SW30: SW_Push_45deg, Button_Switch_Keyboard:SW_Cherry_MX_1.00u_PCB, F.Cu at (338.1, 123.1)
- added SW31: SW_Push_45deg, Button_Switch_Keyboard:SW_Cherry_MX_1.00u_PCB, F.Cu at (338.1, 142.0)
- added SW32: SW_Push_45deg, Button_Switch_Keyboard:SW_Cherry_MX_1.00u_PCB, F.Cu at (338.1, 161.1)
- added SW33: SW_Push_45deg, Button_Switch_Keyboard:SW_Cherry_MX_1.00u_PCB, F.Cu at (338.1, 180.1)
- added SW34: SW_Push_45deg, Button_Switch_Keyboard:SW_Cherry_MX_1.00u_PCB, F.Cu at (357.1, 104.1)
- added SW35: SW_Push_45deg, Button_Switch_Keyboard:SW_Cherry_MX_1.00u_PCB, F.Cu at (357.1, 123.1)
- added SW36: SW_Push_45deg, Button_Switch_Keyboard:SW_Cherry_MX_1.00u_PCB, F.Cu at (357.2, 142.1)
- added SW37: SW_Push_45deg, Button_Switch_Keyboard:SW_Cherry_MX_1.00u_PCB, F.Cu at (357.1, 161.1)
- added SW38: SW_Push_45deg, Button_Switch_Keyboard:SW_Cherry_MX_1.00u_PCB, F.Cu at (357.2, 180.0)
- added SW44: SW_Push_45deg, Button_Switch_Keyboard:SW_Cherry_MX_1.00u_PCB, F.Cu at (59.8, 101.9)
- added SW45: SW_Push_45deg, Button_Switch_Keyboard:SW_Cherry_MX_1.00u_PCB, F.Cu at (78.8, 102.0)
- added SW46: SW_Push_45deg, Button_Switch_Keyboard:SW_Cherry_MX_1.00u_PCB, F.Cu at (97.8, 90.0)
- added SW47: SW_Push_45deg, Button_Switch_Keyboard:SW_Cherry_MX_1.00u_PCB, F.Cu at (116.8, 83.0)
- added SW48: SW_Push_45deg, Button_Switch_Keyboard:SW_Cherry_MX_1.00u_PCB, F.Cu at (135.8, 89.0)
- added SW49: SW_Push_45deg, Button_Switch_Keyboard:SW_Cherry_MX_1.00u_PCB, F.Cu at (154.8, 91.9)
- added SW5: SW_Push_45deg, Button_Switch_Keyboard:SW_Cherry_MX_1.00u_PCB, F.Cu at (262.2, 94.1)
- added SW50: SW_Push_45deg, Button_Switch_Keyboard:SW_Cherry_MX_1.00u_PCB, F.Cu at (59.8, 120.9)
- added SW51: SW_Push_45deg, Button_Switch_Keyboard:SW_Cherry_MX_1.00u_PCB, F.Cu at (78.7, 121.0)
- added SW52: SW_Push_45deg, Button_Switch_Keyboard:SW_Cherry_MX_1.00u_PCB, F.Cu at (97.7, 109.1)
- added SW53: SW_Push_45deg, Button_Switch_Keyboard:SW_Cherry_MX_1.00u_PCB, F.Cu at (116.8, 102.0)
- added SW54: SW_Push_45deg, Button_Switch_Keyboard:SW_Cherry_MX_1.00u_PCB, F.Cu at (135.7, 108.0)
- added SW55: SW_Push_45deg, Button_Switch_Keyboard:SW_Cherry_MX_1.00u_PCB, F.Cu at (154.8, 110.9)
- added SW56: SW_Push_45deg, Button_Switch_Keyboard:SW_Cherry_MX_1.00u_PCB, F.Cu at (59.8, 139.9)
- added SW57: SW_Push_45deg, Button_Switch_Keyboard:SW_Cherry_MX_1.00u_PCB, F.Cu at (78.8, 140.0)
- added SW58: SW_Push_45deg, Button_Switch_Keyboard:SW_Cherry_MX_1.00u_PCB, F.Cu at (97.8, 128.0)
- added SW59: SW_Push_45deg, Button_Switch_Keyboard:SW_Cherry_MX_1.00u_PCB, F.Cu at (116.8, 120.9)
- added SW6: SW_Push_45deg, Button_Switch_Keyboard:SW_Cherry_MX_1.00u_PCB, F.Cu at (262.1, 113.1)
- added SW60: SW_Push_45deg, Button_Switch_Keyboard:SW_Cherry_MX_1.00u_PCB, F.Cu at (135.8, 126.9)
- added SW61: SW_Push_45deg, Button_Switch_Keyboard:SW_Cherry_MX_1.00u_PCB, F.Cu at (154.8, 130.0)
- added SW62: SW_Push_45deg, Button_Switch_Keyboard:SW_Cherry_MX_1.00u_PCB, F.Cu at (59.8, 158.9)
- added SW63: SW_Push_45deg, Button_Switch_Keyboard:SW_Cherry_MX_1.00u_PCB, F.Cu at (78.8, 159.0)
- added SW64: SW_Push_45deg, Button_Switch_Keyboard:SW_Cherry_MX_1.00u_PCB, F.Cu at (97.8, 147.0)
- added SW65: SW_Push_45deg, Button_Switch_Keyboard:SW_Cherry_MX_1.00u_PCB, F.Cu at (116.8, 140.0)
- added SW66: SW_Push_45deg, Button_Switch_Keyboard:SW_Cherry_MX_1.00u_PCB, F.Cu at (135.8, 145.9)
- added SW67: SW_Push_45deg, Button_Switch_Keyboard:SW_Cherry_MX_1.00u_PCB, F.Cu at (154.8, 149.0)
- added SW68: SW_Push_45deg, Button_Switch_Keyboard:SW_Cherry_MX_1.00u_PCB, F.Cu at (59.8, 178.0)
- added SW69: SW_Push_45deg, Button_Switch_Keyboard:SW_Cherry_MX_1.00u_PCB, F.Cu at (78.8, 178.0)
- added SW7: SW_Push_45deg, Button_Switch_Keyboard:SW_Cherry_MX_1.00u_PCB, F.Cu at (262.1, 132.1)
- added SW70: SW_Push_45deg, Button_Switch_Keyboard:SW_Cherry_MX_1.00u_PCB, F.Cu at (97.8, 166.0)
- added SW71: SW_Push_45deg, Button_Switch_Keyboard:SW_Cherry_MX_1.00u_PCB, F.Cu at (116.7, 159.0)
- added SW72: SW_Push_45deg, Button_Switch_Keyboard:SW_Cherry_MX_1.00u_PCB, F.Cu at (135.7, 165.0)
- added SW73: SW_Push_45deg, Button_Switch_Keyboard:SW_Cherry_MX_1.00u_PCB, F.Cu at (154.8, 168.0)
- added SW75: SW_Push_45deg, Button_Switch_Keyboard:SW_Cherry_MX_1.00u_PCB, F.Cu at (174.4, 197.2)
- added SW76: SW_Push_45deg, Button_Switch_Keyboard:SW_Cherry_MX_1.00u_PCB, F.Cu at (152.2, 190.9)
- added SW8: SW_Push_45deg, Button_Switch_Keyboard:SW_Cherry_MX_1.00u_PCB, F.Cu at (262.1, 151.1)
- added SW9: SW_Push_45deg, Button_Switch_Keyboard:SW_Cherry_MX_1.00u_PCB, F.Cu at (262.1, 170.0)
- SW2, SW4: footprint Button_Switch_SMD:Nidec_Copal_CAS-120A -> PTS636_SM43J_SMTR_LFS:SW_PTS636_SM43J_SMTR_LFS
- SW3: footprint Package_SO:SOIC-8_3.9x4.9mm_P1.27mm -> PTS636_SM43J_SMTR_LFS:SW_PTS636_SM43J_SMTR_LFS
- moved D38 447.1 mm to (350.7, 188.6), turned to 90 degrees
- moved D37 439.8 mm to (350.6, 169.6), turned to 90 degrees
- moved D36 433.1 mm to (350.7, 150.5), turned to 90 degrees
- moved D33 427.6 mm to (331.7, 188.7), turned to 90 degrees
- moved D32 420.7 mm to (331.7, 169.6), turned to 90 degrees
- moved D35 420.7 mm to (350.7, 131.6), turned to 90 degrees
- moved D34 416.6 mm to (351.1, 112.8), turned to 90 degrees
- moved D31 414.3 mm to (331.7, 150.5), turned to 90 degrees
- moved D27 412.9 mm to (312.6, 176.6), turned to 90 degrees
- moved D30 408.4 mm to (331.7, 131.4), turned to 90 degrees
- moved D26 405.7 mm to (312.7, 157.5), turned to 90 degrees
- moved D29 403.1 mm to (331.7, 112.7), turned to 90 degrees
- moved D25 398.9 mm to (312.7, 138.7), turned to 90 degrees
- moved D22 393.3 mm to (281.2, 198.4), turned to 90 degrees
- moved D21 392.0 mm to (293.9, 169.6), turned to 90 degrees
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Connections:
- C15 pad 1: GND -> Net-(C15-Pad1)
- C15 pad 2: Net-(C15-Pad2) -> GND
- C25 pad 1: GND -> Net-(C25-Pad1)
- C25 pad 2: Net-(C25-Pad2) -> GND
- R6 pad 2: Net-(C15-Pad2) -> Net-(C15-Pad1)
- R9 pad 2: Net-(C25-Pad2) -> Net-(C25-Pad1)
- Y1 pad 3: Net-(C15-Pad2) -> Net-(C15-Pad1)
- Y2 pad 3: Net-(C25-Pad2) -> Net-(C25-Pad1)
Other:
- board outline added: 317.3 x 144.6 mm
